Commit message: modified sensor color

File: robots/b1_description/xacro/sensors.xacro (robot description, xacro)
@@ -26,5 +26,5 @@
     </link>
     <gazebo reference="lidar_mount">
-        <material>Gazebo/Gray</material>
+        <material>Gazebo/White</material>
     </gazebo>
     <xacro:VLP-16 parent="lidar_mount" name="lidar" topic="/lidar_points"
