Commit message: modified sensors loading

File: robots/b1_description/xacro/robot.xacro (robot description, xacro)
@@ -5,5 +5,4 @@
     <xacro:include filename="$(find b1_description)/xacro/leg.xacro"/>
     <xacro:include filename="$(find b1_description)/xacro/gazebo.xacro"/>
-    <xacro:arg name="SENSORS" default="false"/>
     <!-- Rotor related joint and link is only for demonstrate location. -->
     <!-- Actually, the rotor will rotate and the joint is not fixed. Reduction ratio should be considered. -->
@@ -88,7 +87,15 @@
     <xacro:leg name="RR" mirror="-1" mirror_dae="False"  front_hind="-1" front_hind_dae="False" />
     <xacro:leg name="RL" mirror="1"  mirror_dae="True"   front_hind="-1" front_hind_dae="False" />
+    <!-- Sensors loading -->
+    <xacro:arg name="SENSORS" default="false"/>
+    <xacro:arg name="LIDAR" default="false"/>
+    <xacro:arg name="CAMERAS" default="false"/>
+    <xacro:property name="LIDAR" value="$(arg LIDAR)"/>
+    <xacro:property name="CAMERAS" value="$(arg CAMERAS)"/>
     <xacro:if value="$(arg SENSORS)">
-        <xacro:include filename="$(find b1_description)/xacro/sensors.xacro"/>
+        <xacro:property name="LIDAR" value="true"/>
+        <xacro:property name="CAMERAS" value="true"/>
     </xacro:if>
+    <xacro:include filename="$(find b1_description)/xacro/sensors.xacro"/>
     <!-- <xacro:stairs stairs="15" xpos="0" ypos="2.0" zpos="0" /> -->
 </robot>

File: robots/b1_description/xacro/sensors.xacro (robot description, xacro)
@@ -3,53 +3,62 @@
     <xacro:include filename="$(find velodyne_description)/urdf/VLP-16.urdf.xacro"/>
     <xacro:include filename="$(find b1_description)/xacro/camera/realsense_d435.urdf.xacro" />
-    <material name="gray">
-        <color rgba="0.6 0.6 0.6 1.0"/>
-    </material>
     <!-- Lidar -->
-    <joint name="lidar_mount_joint" type="fixed">
-        <parent link="trunk"/>
-        <child link="lidar_mount"/>
-        <origin xyz="0.16 0 0.11" rpy="0 0 0"/>
-    </joint>
-    <link name="lidar_mount">
-        <visual>
-            <geometry>
-                <box size="0.12 0.12 0.05" />
-            </geometry>
-            <material name="gray"/>
-        </visual>
-        <collision>
-            <geometry>
-                <box size="0.12 0.12 0.05" />
-            </geometry>
-        </collision>
-    </link>
-    <gazebo reference="lidar_mount">
-        <material>Gazebo/White</material>
-    </gazebo>
-    <xacro:VLP-16 parent="lidar_mount" name="lidar" topic="/lidar_points"
-                organize_cloud="true" hz="10" gpu="true">
-        <origin xyz="0 0 0.025" rpy="0 0 0" />
-    </xacro:VLP-16>
+    <xacro:if value="${LIDAR}">
+        <material name="gray">
+            <color rgba="0.6 0.6 0.6 1.0"/>
+        </material>
+        <joint name="lidar_mount_joint" type="fixed">
+            <parent link="trunk"/>
+            <child link="lidar_mount"/>
+            <origin xyz="0.16 0 0.11" rpy="0 0 0"/>
+        </joint>
+        <link name="lidar_mount">
+            <visual>
+                <geometry>
+                    <box size="0.12 0.12 0.05" />
+                </geometry>
+                <material name="gray"/>
+            </visual>
+            <collision>
+                <geometry>
+                    <box size="0.12 0.12 0.05" />
+                </geometry>
+            </collision>
+            <inertial>
+            <mass value="0.00001"/>
+            <origin rpy="0 0 0" xyz="0 0 0"/>
+            <inertia ixx="0.0000001" ixy="0" ixz="0" iyy="0.0000001" iyz="0" izz="0.0000001"/>
+        </inertial>
+        </link>
+        <gazebo reference="lidar_mount">
+            <material>Gazebo/White</material>
+        </gazebo>
+        <xacro:VLP-16 parent="lidar_mount" name="lidar" topic="/lidar_points"
+                    organize_cloud="true" hz="10" gpu="true">
+            <origin xyz="0 0 0.025" rpy="0 0 0" />
+        </xacro:VLP-16>
+    </xacro:if>
     <!-- Cameras -->
-    <!-- Head -->
-    <xacro:realsense_d435 name="d430_head" topics_ns="/d430_head" parent="trunk">
-        <origin xyz="0.46 -0.0075 0.0378" rpy="${PI} 0 0" />
-    </xacro:realsense_d435>
-    <!-- Chin -->
-    <xacro:realsense_d435 name="d430_chin" topics_ns="/d430_chin" parent="trunk">
-        <origin xyz="0.462 -0.0075 -0.06" rpy="${PI} ${PI/2} 0" />
-    </xacro:realsense_d435>
-    <!-- Bottom -->
-    <xacro:realsense_d435 name="d430_bottom" topics_ns="/d430_bottom" parent="trunk">
-        <origin xyz="-0.473 0.0075 -0.065" rpy="0 ${PI/2} 0" />
-    </xacro:realsense_d435>
-    <!-- Left -->
-    <xacro:realsense_d435 name="d430_left" topics_ns="/d430_left" parent="trunk">
-        <origin xyz="-0.095 0.125 -0.0135" rpy="${PI} ${PI/9} ${PI/2}" />
-    </xacro:realsense_d435>
-    <!-- Right -->
-    <xacro:realsense_d435 name="d435" topics_ns="/d435_right" parent="trunk">
-        <origin xyz="-0.1025 -0.1175 -0.0375" rpy="0 ${PI/9} -${PI/2}" />
-    </xacro:realsense_d435>
+    <xacro:if value="${CAMERAS}">
+        <!-- Head -->
+        <xacro:realsense_d435 name="d430_head" topics_ns="/d430_head" parent="trunk">
+            <origin xyz="0.46 -0.0075 0.0378" rpy="${PI} 0 0" />
+        </xacro:realsense_d435>
+        <!-- Chin -->
+        <xacro:realsense_d435 name="d430_chin" topics_ns="/d430_chin" parent="trunk">
+            <origin xyz="0.462 -0.0075 -0.06" rpy="${PI} ${PI/2} 0" />
+        </xacro:realsense_d435>
+        <!-- Bottom -->
+        <xacro:realsense_d435 name="d430_bottom" topics_ns="/d430_bottom" parent="trunk">
+            <origin xyz="-0.473 0.0075 -0.065" rpy="0 ${PI/2} 0" />
+        </xacro:realsense_d435>
+        <!-- Left -->
+        <xacro:realsense_d435 name="d430_left" topics_ns="/d430_left" parent="trunk">
+            <origin xyz="-0.095 0.125 -0.0135" rpy="${PI} ${PI/9} ${PI/2}" />
+        </xacro:realsense_d435>
+        <!-- Right -->
+        <xacro:realsense_d435 name="d435" topics_ns="/d435_right" parent="trunk">
+            <origin xyz="-0.1025 -0.1175 -0.0375" rpy="0 ${PI/9} -${PI/2}" />
+        </xacro:realsense_d435>
+    </xacro:if>
 </robot>
